File: gyro_board/gyro_board.brd (EAGLE design)
At the start: 53.8 x 24.4 mm, 22 parts, among them IC1 LM2937, Q1 BSS123, Q2 BSS123, U1 VL53L0X

Commit message: board
Connections:
- net GND: now also LSM6DS0TR.P$4
Routing:
- net GND: track 110.9 -> 112.6 mm, vias 6 -> 7
Other:
- board text added: "GYRO"
- board text added: "LASER"
- board text removed: "MISO"
Changed lines of the file:
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@@
 <text x="66.548" y="4.064" size="1.27" layer="25" rot="R90">SCK</text>
 <text x="69.088" y="4.064" size="1.143" layer="25" rot="R90">MOSI</text>
-<text x="71.628" y="4.064" size="1.143" layer="25" rot="R90">MISO</text>
 <rectangle x1="16.256" y1="72.898" x2="31.75" y2="104.14" layer="30"/>
 <rectangle x1="76.962" y1="72.898" x2="92.456" y2="104.14" layer="30"/>
@@
 <wire x1="35.306" y1="4.064" x2="35.306" y2="20.32" width="0" layer="20"/>
 <wire x1="73.406" y1="4.064" x2="73.406" y2="20.32" width="0" layer="20"/>
+<text x="60.198" y="8.636" size="1.778" layer="25" rot="R90">GYRO</text>
+<text x="58.674" y="17.526" size="1.778" layer="25">LASER</text>
 </plain>
 <attributes>
@@
 <attribute name="VALUE" x="46.99" y="5.715" size="1.27" layer="27" rot="R180"/>
 </element>
-<element name="Q1" library="transistor-small-signal" package="SOT23" value="BSS123" x="64.262" y="7.874" rot="R180"/>
-<element name="Q2" library="transistor-small-signal" package="SOT23" value="BSS123" x="68.326" y="7.874" rot="R180"/>
-<element name="R1" library="resistor" package="R0805" value="10k" x="64.262" y="10.922"/>
-<element name="R2" library="resistor" package="R0805" value="10k" x="68.58" y="11.176"/>
-<element name="R3" library="resistor" package="R0805" value="10k" x="61.722" y="9.652" rot="R90"/>
-<element name="R4" library="resistor" package="R0805" value="10k" x="71.628" y="9.906" rot="R90"/>
-<element name="IC1" library="linear" package="TO263-3" value="LM2937" x="41.402" y="16.002"/>
-<element name="C1" library="resistor" package="C0805K" value="100n" x="39.116" y="7.874"/>
-<element name="C2" library="resistor" package="C0805K" value="10uF" x="39.116" y="6.096"/>
-<element name="C3" library="resistor" package="C0805K" value="100n" x="43.18" y="7.874" rot="R180"/>
-<element name="C4" library="resistor" package="C0805K" value="10uF" x="43.18" y="6.096" rot="R180"/>
-<element name="LSM6DS0TR" library="main" package="LGA16L" value="L3GD20H" x="54.102" y="10.16" rot="R90"/>
-<element name="C5" library="resistor" package="C0805K" value="10n" x="50.546" y="11.176" rot="R90"/>
-<element name="C6" library="resistor" package="C0805K" value="100n" x="56.896" y="9.652" rot="R90"/>
-<element name="U1" library="VL53L0X" package="VL53L0X" value="VL53L0X" x="54.61" y="17.78" rot="R90"/>
-<element name="R5" library="resistor" package="R0805" value="10k" x="55.372" y="20.32"/>
-<element name="C7" library="resistor" package="C0805K" value="10uF" x="51.054" y="17.78" rot="R90"/>
+<element name="Q1" library="transistor-small-signal" package="SOT23" value="BSS123" x="64.262" y="7.874" smashed="yes" rot="R180">
+<attribute name="VALUE" x="66.167" y="11.049" size="1.27" layer="27" rot="R180"/>
+</element>
+<element name="Q2" library="transistor-small-signal" package="SOT23" value="BSS123" x="68.326" y="7.874" smashed="yes" rot="R180">
+<attribute name="VALUE" x="70.231" y="11.049" size="1.27" layer="27" rot="R180"/>
+</element>
+<element name="R1" library="resistor" package="R0805" value="10k" x="64.262" y="10.922" smashed="yes">
+<attribute name="VALUE" x="63.5" y="8.636" size="1.27" layer="27"/>
+</element>
+<element name="R2" library="resistor" package="R0805" value="10k" x="68.58" y="11.176" smashed="yes">
+<attribute name="VALUE" x="67.818" y="8.89" size="1.27" layer="27"/>
+</element>
+<element name="R3" library="resistor" package="R0805" value="10k" x="61.722" y="9.652" smashed="yes" rot="R90">
+<attribute name="VALUE" x="64.008" y="8.89" size="1.27" layer="27" rot="R90"/>
+</element>
+<element name="R4" library="resistor" package="R0805" value="10k" x="71.628" y="9.906" smashed="yes" rot="R90">
+<attribute name="VALUE" x="73.914" y="9.144" size="1.27" layer="27" rot="R90"/>
+</element>
+<element name="IC1" library="linear" package="TO263-3" value="LM2937" x="41.402" y="16.002" smashed="yes">
+<attribute name="VALUE" x="48.26" y="10.414" size="1.27" layer="27" rot="R90"/>
+</element>
+<element name="C1" library="resistor" package="C0805K" value="100n" x="39.116" y="7.874" smashed="yes">
+<attribute name="VALUE" x="38.116" y="5.974" size="1.016" layer="27"/>
+</element>
+<element name="C2" library="resistor" package="C0805K" value="10uF" x="39.116" y="6.096" smashed="yes">
+<attribute name="VALUE" x="38.116" y="4.196" size="1.016" layer="27"/>
+</element>
+<element name="C3" library="resistor" package="C0805K" value="100n" x="43.18" y="7.874" smashed="yes" rot="R180">
+<attribute name="VALUE" x="44.18" y="9.774" size="1.016" layer="27" rot="R180"/>
+</element>
+<element name="C4" library="resistor" package="C0805K" value="10uF" x="43.18" y="6.096" smashed="yes" rot="R180">
+<attribute name="VALUE" x="44.18" y="7.996" size="1.016" layer="27" rot="R180"/>
+</element>
+<element name="LSM6DS0TR" library="main" package="LGA16L" value="L3GD20H" x="54.102" y="10.16" smashed="yes" rot="R90"/>
+<element name="C5" library="resistor" package="C0805K" value="10n" x="50.546" y="11.176" smashed="yes" rot="R90">
+<attribute name="VALUE" x="52.446" y="10.176" size="1.016" layer="27" rot="R90"/>
+</element>
+<element name="C6" library="resistor" package="C0805K" value="100n" x="56.896" y="9.652" smashed="yes" rot="R90">
+<attribute name="VALUE" x="58.796" y="8.652" size="1.016" layer="27" rot="R90"/>
+</element>
+<element name="U1" library="VL53L0X" package="VL53L0X" value="VL53L0X" x="54.61" y="17.78" smashed="yes" rot="R90"/>
+<element name="R5" library="resistor" package="R0805" value="10k" x="55.372" y="20.32" smashed="yes">
+<attribute name="VALUE" x="54.61" y="18.034" size="1.27" layer="27"/>
+</element>
+<element name="C7" library="resistor" package="C0805K" value="10uF" x="51.054" y="17.78" smashed="yes" rot="R90">
+<attribute name="VALUE" x="52.954" y="16.78" size="1.016" layer="27" rot="R90"/>
+</element>
 <element name="U$1" library="fiducial" package="CIRCLE-1MM-2R" value="" x="68.58" y="22.352"/>
 <element name="U$2" library="fiducial" package="CIRCLE-1MM-2R" value="" x="34.544" y="22.098"/>
@@
 <wire x1="56.888" y1="10.66" x2="56.896" y2="10.652" width="0.3048" layer="1"/>
 <wire x1="52.802" y1="10.16" x2="53.848" y2="10.16" width="0.3048" layer="1"/>
-<wire x1="53.848" y1="10.16" x2="54.356" y2="10.668" width="0.3048" layer="1"/>
+<wire x1="53.848" y1="10.16" x2="54.102" y2="10.414" width="0.3048" layer="1"/>
+<wire x1="54.102" y1="10.414" x2="54.356" y2="10.668" width="0.3048" layer="1"/>
 <wire x1="54.356" y1="10.668" x2="55.394" y2="10.668" width="0.3048" layer="1"/>
 <wire x1="55.394" y1="10.668" x2="55.402" y2="10.66" width="0.3048" layer="1"/>
@@
 <vertex x="8.636" y="-8.128"/>
 </polygon>
-<via x="58.674" y="12.7" extent="1-16" drill="0.6"/>
+<via x="57.404" y="13.208" extent="1-16" drill="0.6"/>
 <via x="59.944" y="20.828" extent="1-16" drill="0.6"/>
 <via x="71.12" y="21.336" extent="1-16" drill="0.6"/>
@@
 </polygon>
 <via x="49.022" y="8.128" extent="1-16" drill="0.6"/>
+<contactref element="LSM6DS0TR" pad="P$4"/>
+<wire x1="54.602" y1="8.86" x2="54.602" y2="9.914" width="0.254" layer="1"/>
+<wire x1="54.602" y1="9.914" x2="54.102" y2="10.414" width="0.254" layer="1"/>
+<via x="67.056" y="4.826" extent="1-16" drill="0.6"/>
 </signal>
 <signal name="+5V">
