File: gyro_board/gyro_board.sch (EAGLE design)
At the start: 19 parts, among them IC1 LM2937, Q1 BSS123, Q2 BSS123, U1 VL53L0X

Commit message: board
Connections:
- net GND: now also LSM6DS0TR.SDO
Changed lines of the file:
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@@
 <part name="+3V10" library="supply1" deviceset="+3V3" device=""/>
 <part name="GND12" library="supply1" deviceset="GND" device=""/>
+<part name="GND13" library="supply1" deviceset="GND" device=""/>
 </parts>
 <sheets>
@@
 <attribute name="VALUE" x="253.238" y="162.052" size="1.27" layer="96" rot="R90"/>
 </instance>
+<instance part="GND13" gate="1" x="149.86" y="149.86" smashed="yes">
+<attribute name="VALUE" x="146.812" y="148.082" size="1.27" layer="96"/>
+</instance>
 </instances>
 <busses>
@@
 <wire x1="243.84" y1="165.1" x2="248.92" y2="165.1" width="0.1524" layer="91"/>
 </segment>
+<segment>
+<pinref part="LSM6DS0TR" gate="G$1" pin="SDO"/>
+<pinref part="GND13" gate="1" pin="GND"/>
+<wire x1="154.94" y1="154.94" x2="149.86" y2="154.94" width="0.1524" layer="91"/>
+<wire x1="149.86" y1="154.94" x2="149.86" y2="152.4" width="0.1524" layer="91"/>
+</segment>
 </net>
